File: kicad/lora-v2.kicad_sch (KiCad schematic)
At the start: 48 parts, among them J1 USB_C_Receptacle_USB2.0_16P, SW1 bootsl, SW2 reset, U1 RP2040, U2 SX1262IMLTRT, U3 4259-63, U4 AP2112K-3.3TRG1, U5 W25Q16JVSS, Y1 32MHz, Y2 12MHz

Commit message: message
Parts:
- added C26, C27: 12pF, Capacitor_SMD:C_0402_1005Metric, symbol Device:C
- added C28: 10uF, Capacitor_SMD:C_0402_1005Metric, symbol Device:C
- added R8: 10k, Resistor_SMD:R_0402_1005Metric, symbol Device:R
Connections:
- net +3V3: now also C28.1, R8.1
- net Earth: now also FL1.10 (GND), FL1.2 (GND), FL1.5 (GND), FL1.7 (GND), FL1.9 (GND), U1.19 (TESTEN), C26.1, C27.1, C28.2
- net SX_DIO2: now also R1.2; no longer R1.1
- net SX_NSS: now also R8.2
- net SX_XTA: now also C26.2
- net SX_XTB: now also C27.2
- net at U3.4 (CTRL): now also C6.1, R1.1; no longer C7.1
- new net: C7.1, U3.5 (RFC)
Other:
- moved on the sheet: C7, Y1
