File: kicad/lora-v2.kicad_sch (KiCad schematic)
At the start: 52 parts, among them J1 USB_C_Receptacle_USB2.0_16P, SW1 bootsl, SW2 reset, U1 RP2040, U2 SX1262IMLTRT, U3 4259-63, U4 AP2112K-3.3TRG1, U5 W25Q16JVSS, Y1 32MHz, Y2 12MHz

Commit message: added
Parts:
- added J2: Conn_01x04, Connector_PinHeader_2.54mm:PinHeader_1x04_P2.54mm_Vertical, symbol Connector_Generic:Conn_01x04
Connections:
- net +3V3: now also J2.1 (Pin_1)
- net SDA: now reaches U1.6 (GPIO4)
- net SDA: now also J2.3 (Pin_3)
- net SCL: now reaches U1.7 (GPIO5)
- net SCL: now also J2.2 (Pin_2)
- new net GND: J2.4 (Pin_4)
- no-connect marks 28 -> 26
